File: FEHLERboard.kicad_pcb (KiCad board)
At the start: 2 copper layers, 100 parts, among them J1 Conn_01x01, J10 Conn_01x01, J11 Conn_01x01, J12 Conn_01x01, J13 Conn_01x01, J14 Conn_01x01, J15 Conn_01x01, J16 Conn_01x01, J17 Conn_01x01, J18 Conn_01x01, J19 USB_B_Micro, J2 Conn_01x01, J20 Conn_01x01, J21 Conn_01x01, J22 Conn_01x01, J23 USB_B_Micro, J24 Conn_01x01, J25 Conn_01x01, J26 Conn_01x01, J27 Conn_01x01, J28 Conn_01x01, J29 Conn_01x01, J3 Conn_01x01, J30 Conn_01x01, J31 Conn_01x01, J32 Conn_01x01, J33 Conn_01x01, J34 Conn_01x01, J35 Conn_01x01, J36 Conn_01x01, J37 Conn_01x01, J38 Conn_01x01, J39 Conn_01x01, J4 Conn_01x01, J40 Conn_01x01, J41 Conn_01x01, J42 Conn_01x01, J43 Conn_01x01, J5 Conn_01x01, J6 Conn_01x01, J7 Conn_01x01, J8 Conn_01x01, J9 Conn_01x01, Q1 Q_NPN_BEC, Q2 Q_NPN_BEC, Q3 Q_NPN_BEC, Q4 Q_NPN_BEC, U1 ESP32-WROOM-32, U2 ESP32-WROOM-32, U3 MT3420C, U4 MT3420C, U5 TCAN330, U6 TCAN330, U7 CH340K, U8 CH340K

Commit message: Failure upgrade V2
Parts:
- added G***: LOGO, TheBrutzlers_Lib:Platinenmacher_14, F.Cu at (172.1, 86.7)
- added G***: LOGO, TheBrutzlers_Lib:Symbol_kurzschlussblog_20mm, F.Cu at (155.2, 146.7)
- added G***: LOGO, TheBrutzlers_Lib:thebrutzler_approved_small02, F.Cu at (158.0, 105.4)
- added G***: LOGO, TheBrutzlers_Lib:Symbol_kurzschlussblog_20mm, B.Cu at (159.3, 146.7)
- added G***: LOGO, TheBrutzlers_Lib:Platinenmacher_14, B.Cu at (172.1, 86.7)
- added G***: LOGO, TheBrutzlers_Lib:thebrutzler_approved_small02, B.Cu at (158.0, 105.4)
- added J35: Conn_01x01, TestPoint:TestPoint_THTPad_1.5x1.5mm_Drill0.7mm, F.Cu at (174.2, 125.0)
- added J44: Conn_01x01, TestPoint:TestPoint_THTPad_D1.5mm_Drill0.7mm, F.Cu at (148.5, 128.8)
- added J45: Conn_01x01, TestPoint:TestPoint_THTPad_D1.5mm_Drill0.7mm, F.Cu at (146.0, 137.5)
- added J46: Conn_01x01, TestPoint:TestPoint_THTPad_1.5x1.5mm_Drill0.7mm, F.Cu at (165.5, 76.2)
- added J47: Conn_01x01, TestPoint:TestPoint_THTPad_1.5x1.5mm_Drill0.7mm, F.Cu at (181.2, 110.2)
- added J48: Conn_01x01, TestPoint:TestPoint_THTPad_1.5x1.5mm_Drill0.7mm, F.Cu at (110.5, 79.2)
- added J49: Conn_01x01, TestPoint:TestPoint_THTPad_1.5x1.5mm_Drill0.7mm, F.Cu at (119.2, 117.0)
- added J50: Conn_01x01, TestPoint:TestPoint_THTPad_1.5x1.5mm_Drill0.7mm, F.Cu at (126.8, 140.8)
- added J51: Conn_01x01, TestPoint:TestPoint_THTPad_1.5x1.5mm_Drill0.7mm, F.Cu at (178.5, 151.0)
- added J52: Conn_01x01, TestPoint:TestPoint_THTPad_1.5x1.5mm_Drill0.7mm, F.Cu at (127.5, 102.2)
- added J53: Conn_01x01, TestPoint:TestPoint_THTPad_1.5x1.5mm_Drill0.7mm, F.Cu at (139.5, 80.2)
- added J54: Conn_01x01, TestPoint:TestPoint_THTPad_1.5x1.5mm_Drill0.7mm, F.Cu at (154.2, 78.5)
- added R29: 4K7, Resistor_SMD:R_0603_1608Metric, F.Cu at (148.5, 131.5)
- added R30: 4K7, Resistor_SMD:R_0603_1608Metric, F.Cu at (146.0, 134.8)
- added R31: 4K7, Resistor_SMD:R_0603_1608Metric, F.Cu at (115.8, 124.5)
- added R32: 4K7, Resistor_SMD:R_0603_1608Metric, F.Cu at (184.2, 85.2)
- moved C6 132.7 mm to (171.0, 130.0), turned to -90 degrees
- moved J39 119.1 mm to (187.0, 80.2)
- moved J32 111.8 mm to (187.0, 77.8)
- moved J5 104.1 mm to (184.5, 122.5)
- moved J8 101.1 mm to (173.5, 127.8)
- moved J6 98.8 mm to (184.5, 120.0)
- moved J14 97.9 mm to (187.0, 82.8)
- moved C13 96.4 mm to (143.5, 96.5)
- moved J17 91.9 mm to (154.2, 81.0)
- moved C11 91.0 mm to (139.0, 90.8), turned to 90 degrees
- moved R25 90.1 mm to (139.8, 124.8)
- moved R22 89.4 mm to (185.0, 76.5), turned to 90 degrees
- moved J11 88.7 mm to (184.5, 80.2)
- moved J10 88.7 mm to (184.5, 82.8)
- moved J12 88.3 mm to (187.0, 85.2)
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Connections:
- C12 pad 1: +5V -> +5F
- U8 pad 7: +5V -> +5F
Routing:
- net +3V3: track 26.2 -> 279.9 mm, vias 2 -> 14
- net /SPI_CLK: track 0.00 -> 96.2 mm, vias 0 -> 2
- net /CAN-: track 0.00 -> 89.5 mm
- net /CAN+: track 0.00 -> 87.4 mm
- net /UART2_TX: track 0.00 -> 86.2 mm, vias 0 -> 1
- net /UART2_RX: track 0.00 -> 83.4 mm, vias 0 -> 1
- net GND: track 40.1 -> 109.5 mm, vias 27 -> 112
- net +5V: track 34.4 -> 101.1 mm, vias 1 -> 3
- net /TX: track 51.7 -> 110.5 mm
- net +5F: track 41.3 -> 92.4 mm, vias 2 -> 4
- net /UART2_TX_FAIL: track 69.2 -> 88.0 mm, vias 3 -> 5
- net /UART2_RX_FAIL: track 67.5 -> 81.7 mm
- net Net-(J15-Pad1): track 0.00 -> 9.68 mm
- net Net-(Q3-Pad2): track 4.45 -> 10.1 mm, vias 0 -> 2
- net Net-(Q3-Pad1): track 0.00 -> 5.01 mm
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- added copper zone on F.Cu, net +3V3
- added copper zone on F.Cu, net /CAP_TOUCH
- added copper zone on F.Cu, net /CAP_TOUCH_FAIL
- added copper zone on B.Cu, net GND
- removed copper zone on B.Cu, net /CAP_TOUCH_FAIL
Other:
- board outline added: 99 x 84.5 mm
- board text added: "+5V FAIL"
- board text added: "3V3"
- board text added: "3V3_FAIL"
- board text added: "5V"
- board text added: "ADC"
- board text added: "ADC_FAIL"
- board text added: "AzuBi-Board"
- board text added: "CAN+"
- board text added: "CAN+ FAIL"
- board text added: "CAN-"
- board text added: "CAN- FAIL"
- board text added: "CAN_RX"
- board text added: "FB"
- board text added: "FB_FAIL"
- board text added: "RX"
- board text added: "RX_FAIL"
- board text added: "SPI CLK"
- board text added: "SPI CLK FAIL"
- board text added: "TX FAIL"
- board text added: "UART2 RX"
- board text added: "UART2 TX"
- board text added: "UART_2 RX_FAIL"
- board text added: "UART_2 TX_FAIL"
- board text added: "USB+"
- board text added: "USB+ FAIL"
- board text added: "USB-"
- board text added: "USB- FAIL"
