File: FEHLERboard.kicad_sch (KiCad schematic)
At the start: 99 parts, among them J1 Conn_01x01, J10 Conn_01x01, J11 Conn_01x01, J12 Conn_01x01, J13 Conn_01x01, J14 Conn_01x01, J15 Conn_01x01, J16 Conn_01x01, J17 Conn_01x01, J18 Conn_01x01, J19 USB_B_Micro, J2 Conn_01x01, J20 Conn_01x01, J21 Conn_01x01, J22 Conn_01x01, J23 USB_B_Micro, J24 Conn_01x01, J25 Conn_01x01, J26 Conn_01x01, J27 Conn_01x01, J28 Conn_01x01, J29 Conn_01x01, J3 Conn_01x01, J30 Conn_01x01, J31 Conn_01x01, J32 Conn_01x01, J33 Conn_01x01, J34 Conn_01x01, J35 Conn_01x01, J36 Conn_01x01, J37 Conn_01x01, J38 Conn_01x01, J39 Conn_01x01, J4 Conn_01x01, J40 Conn_01x01, J41 Conn_01x01, J42 Conn_01x01, J43 Conn_01x01, J5 Conn_01x01, J6 Conn_01x01, J7 Conn_01x01, J8 Conn_01x01, J9 Conn_01x01, Q1 Q_NPN_BEC, Q2 Q_NPN_BEC, Q3 Q_NPN_BEC, Q4 Q_NPN_BEC, U1 ESP32-WROOM-32, U2 ESP32-WROOM-32, U3 MT3420C, U4 MT3420C, U5 TCAN330, U6 TCAN330, U7 CH340K, U8 CH340K

Commit message: Failure upgrade V2
Parts:
- added J44, J45: Conn_01x01, TestPoint:TestPoint_THTPad_D1.5mm_Drill0.7mm, symbol Connector_Generic:Conn_01x01
- added J46, J47, J48, J49, J50, J51, J52, J53, J54: Conn_01x01, TestPoint:TestPoint_THTPad_1.5x1.5mm_Drill0.7mm, symbol Connector_Generic:Conn_01x01
- added R29, R30, R31, R32: 4K7, Resistor_SMD:R_0603_1608Metric, symbol Device:R
Connections:
- net +5F: now also C12.1, U8.7 (VCC)
- net +5V: no longer C12.1, U8.7 (VCC)
- net GND: now also J46.1 (Pin_1), J47.1 (Pin_1), J48.1 (Pin_1), J49.1 (Pin_1), J50.1 (Pin_1), J51.1 (Pin_1), J52.1 (Pin_1), J53.1 (Pin_1), J54.1 (Pin_1), R31.2, R32.2
- net SPI_CLK: now also R32.1
- net SPI_CLK_FAIL: now also R31.1
- net USB+_FAIL: now also R30.2
- net USB-_FAIL: now also R29.2
- new net: J44.1 (Pin_1), R29.1
- new net: J45.1 (Pin_1), R30.1
